Commit message: oscar has a simulator

File: oscar/oscar_description/urdf/oscar.urdf.xacro (robot description, xacro)
@@ -1,26 +1,28 @@
 <?xml version="1.0"?>
 <robot name="oscar" xmlns:xacro="http://www.ros.org/wiki/xacro">
-  <xacro:property name="PI" value="3.1415926535897931" />
-  <xacro:property name="chassis_length" value="0.12" />
+  <xacro:property name="chassis_length" value="0.08" />
   <xacro:property name="chassis_width"  value="0.065" />
   <xacro:property name="chassis_height" value="0.01" />
-  <xacro:property name="chassis_mass"   value="0.18" />
+  <xacro:property name="chassis_mass"   value="0.20" />
   <xacro:property name="chassis_dx"     value="0.04" />
   <xacro:property name="left_wheel_radius"  value="0.03" />
   <xacro:property name="right_wheel_radius" value="0.03" />
-  <xacro:property name="wheel_width"  value="0.01" />
+  <xacro:property name="wheel_width"  value="0.02" />
   <xacro:property name="wheel_track"  value="0.09" />
-  <xacro:property name="wheel_mass"   value="0.01" />
-  <xacro:property name="wheel_joint_damping" value="0.01" />
-  <xacro:property name="wheel_joint_friction" value="0.01" />
+  <xacro:property name="wheel_mass"   value="0.02" />
+  <xacro:property name="steering_servo_no_load_speed" value="2.5" />
+  <xacro:property name="rear_wheel_axle_joint_eff_limit" value="10.0" />
+  <xacro:property name="rear_wheel_axle_joint_vel_limit" value="20.0" />
+  <xacro:property name="rear_wheel_joint_damping"  value="0.01" />
+  <xacro:property name="rear_wheel_joint_friction" value="0.01" />
   <xacro:property name="front_wheel_radius"  value="0.03" />
   <xacro:property name="front_wheel_L"       value="0.08" />
-  <xacro:property name="front_wheel_width"   value="0.01" />
-  <xacro:property name="steering_servo_stall_torque" value="1.0" />
-  <xacro:property name="steering_servo_no_load_speed" value="5.0" />
-  <xacro:property name="front_wheel_axle_joint_eff_limit" value="5.0" />
-  <xacro:property name="front_wheel_axle_joint_vel_limit" value="5.0" />
-  <xacro:property name="front_wheel_axle_joint_damping" value="0.01" />
-  <xacro:property name="front_wheel_axle_joint_friction" value="0.01" />
+  <xacro:property name="front_wheel_width"   value="0.02" />
+  <xacro:property name="steering_servo_stall_torque" value="10.0" />
+  <xacro:property name="steering_servo_no_load_speed" value="2.5" />
+  <xacro:property name="front_wheel_axle_joint_eff_limit" value="10.0" />
+  <xacro:property name="front_wheel_axle_joint_vel_limit" value="20.0" />
+  <xacro:property name="front_wheel_axle_joint_damping"  value="0.00001" />
+  <xacro:property name="front_wheel_axle_joint_friction" value="0.00001" />
   <!-- Inertia macros -->
   <xacro:include filename="$(find common_robots)/urdf/inertias.urdf.xacro" />
@@ -36,4 +38,8 @@
       <material name="transp_green"/>
     </visual>
+    <!-- <collision> -->
+    <!--   <origin xyz="${chassis_dx} 0.00  0.00" rpy="0 0 0"/> -->
+    <!--   <geometry><box size="${chassis_length} ${chassis_width} ${chassis_height}"/></geometry> -->
+    <!-- </collision> -->
     <xacro:inertial_cuboid_with_pose mass="${chassis_mass}" x_length="${chassis_length}" y_length="${chassis_width}" z_length="${chassis_height}">
       <origin xyz="${chassis_dx} 0.00  0.00" rpy="0 0 0"/>
@@ -55,3 +61,12 @@
     <origin xyz="${front_wheel_L} 0 0" rpy="0 0 0" />
   </xacro:front_wheel>
+  <!-- Sensors -->
+  <link name="imu_link">
+    <visual><geometry><sphere radius="0.0025"/></geometry></visual>
+  </link>
+  <joint name="imu_joint" type="fixed">
+    <origin xyz="0 0 0" rpy="0 0 0" />
+    <parent link="base_link" />
+    <child link="imu_link" />
+  </joint>
 </robot>

File: oscar/oscar_description/urdf/oscar_v0.urdf.xacro (robot description, xacro)
@@ -1,7 +1,5 @@
 <?xml version="1.0"?>
 <robot name="oscar" xmlns:xacro="http://www.ros.org/wiki/xacro">
-  <xacro:property name="high_definition_wheel_visual" value="true" />
+  <xacro:property name="high_definition_wheel_visual" value="True" />
   <xacro:include filename="$(find oscar_description)/urdf/oscar.urdf.xacro" />
-  <!-- Bring in simulation data for Gazebo. -->
-  <xacro:include filename="$(find oscar_description)/urdf/oscar.gazebo" />
 </robot>

File: oscar/oscar_description/urdf/wheels.urdf.xacro (robot description, xacro)
@@ -28,14 +28,14 @@
       <xacro:insert_block name="joint_pose" />
       <axis xyz="0 1 0" />
-      <dynamics damping="${wheel_joint_damping}" friction="${wheel_joint_friction}"/>
-      <limit effort="1" velocity="10"/>
+      <dynamics damping="${rear_wheel_joint_damping}" friction="${rear_wheel_joint_friction}"/>
+      <limit effort="${rear_wheel_axle_joint_eff_limit}" velocity="${rear_wheel_axle_joint_vel_limit}"/>
     </joint>
     <transmission name="${prefix}_wheel_trans">
       <type>transmission_interface/SimpleTransmission</type>
       <joint name="${prefix}_wheel_joint">
-	<hardwareInterface>hardware_interface/VelocityJointInterface</hardwareInterface>
+	<hardwareInterface>hardware_interface/EffortJointInterface</hardwareInterface>
       </joint>
       <actuator name="${prefix}_actuator">
-        <hardwareInterface>VelocityJointInterface</hardwareInterface>
+        <hardwareInterface>EffortJointInterface</hardwareInterface>
 	<mechanicalReduction>1</mechanicalReduction>
       </actuator>
@@ -49,4 +49,11 @@
         <geometry><cylinder radius="0.0025" length="0.01"/></geometry>
       </visual>
+      <!--<collision>
+	<origin xyz="0 0 0"/>
+        <geometry><cylinder radius="0.0025" length="0.01"/></geometry>
+      </collision>-->
+      <xacro:inertial_cylinder_with_pose mass="0.01" radius="0.0025" height="0.01">
+	<origin xyz="0 0 0"/>
+      </xacro:inertial_cylinder_with_pose>
     </link>
     <joint name="steering_link_joint" type="fixed">
@@ -57,8 +64,15 @@
     <link name="front_axle_carrier_link">
       <visual>
-        <origin xyz="0 0 0"/>
+        <origin xyz="0 0 0" rpy="${pi/2} 0 0 "/>
         <geometry><cylinder radius="0.0025" length="0.01"/></geometry>
         <material name="yellow" />
       </visual>
+      <!--<collision>
+	 <origin xyz="0 0 0" rpy="${pi/2} 0 0"/>
+         <geometry><cylinder radius="0.0025" length="0.01"/></geometry>
+      </collision>-->
+      <xacro:inertial_cylinder_with_pose mass="0.01" radius="0.0025" height="0.01">
+	<origin xyz="0 0 0" rpy="${pi/2} 0 0"/>
+      </xacro:inertial_cylinder_with_pose>
     </link>
     <joint name="steering_joint" type="revolute">
@@ -69,6 +83,20 @@
       <limit lower="${-pi/4}" upper="${pi/4}" effort="${steering_servo_stall_torque}" velocity="${steering_servo_no_load_speed}"/>
     </joint>
+    <transmission name="steering_trans">
+      <type>transmission_interface/SimpleTransmission</type>
+      <joint name="steering_joint">
+    	<hardwareInterface>hardware_interface/PositionJointInterface</hardwareInterface>
+      </joint>
+      <actuator name="steering_act">
+        <mechanicalReduction>1</mechanicalReduction>
+      </actuator>
+    </transmission>
     <link name="front_wheel_link">
       <visual>
+	<xacro:if value="${high_definition_wheel_visual}">
+	  <xacro:property name="wheel_mesh_scale" value="${front_wheel_radius/0.03}" scope="local"/>
+	  <origin xyz="0 0 0" rpy="0 0 ${pi/2}"/>
+          <geometry><mesh scale="1. ${wheel_mesh_scale} ${wheel_mesh_scale}" filename="package://common_robots/meshes/wheel_60.dae"/></geometry>
+	</xacro:if>
 	<xacro:unless value="${high_definition_wheel_visual}">
 	  <origin xyz="0 0 0" rpy="${pi/2} 0 0"/>
@@ -76,10 +104,12 @@
           <material name="transp_yellow" />
 	</xacro:unless>
-	<xacro:if value="${high_definition_wheel_visual}">
-	  <xacro:property name="wheel_mesh_scale" value="${wheel_radius/0.03}" />
-	  <origin xyz="0 0 0" rpy="0 0 ${pi/2}"/>
-          <geometry><mesh scale="1. ${wheel_mesh_scale} ${wheel_mesh_scale}" filename="package://common_robots/meshes/wheel_60.dae"/></geometry>
-	</xacro:if>
       </visual>
+      <collision>
+        <origin xyz="0 0 0" rpy="${pi/2} 0 0"/>
+        <geometry><cylinder radius="${front_wheel_radius}" length="${front_wheel_width}"/></geometry>
+      </collision>
+      <xacro:inertial_cylinder_with_pose mass="${wheel_mass}" radius="${front_wheel_radius}" height="${front_wheel_width}">
+	<origin xyz="0 0 0" rpy="${pi/2} 0 0"/>
+      </xacro:inertial_cylinder_with_pose>
     </link>
     <joint name="front_axle_joint" type="continuous">
@@ -90,4 +120,14 @@
       <dynamic damping="${front_wheel_axle_joint_damping}" friction="{front_wheel_axle_joint_friction}"/>
     </joint>
+    <transmission name="font_wheel_trans">
+      <type>transmission_interface/SimpleTransmission</type>
+      <joint name="front_axle_joint">
+	<hardwareInterface>hardware_interface/EffortJointInterface</hardwareInterface>
+      </joint>
+      <actuator name="front_axle__actuator">
+        <hardwareInterface>EffortJointInterface</hardwareInterface>
+	<mechanicalReduction>1</mechanicalReduction>
+      </actuator>
+    </transmission>
   </xacro:macro>
 </robot>

Commit message: simulation

File: oscar/oscar_description/urdf/oscar.urdf.xacro (robot description, xacro)
@@ -25,7 +25,8 @@
   <xacro:property name="front_wheel_axle_joint_damping"  value="0.00001" />
   <xacro:property name="front_wheel_axle_joint_friction" value="0.00001" />
-  <!-- Inertia macros -->
+  <!-- Common macros -->
   <xacro:include filename="$(find common_robots)/urdf/inertias.urdf.xacro" />
   <xacro:include filename="$(find common_robots)/urdf/materials.urdf" />
+  <xacro:include filename="$(find common_robots)/urdf/sensors.urdf.xacro" />
   <!-- Car Parts -->
   <xacro:include filename="$(find oscar_description)/urdf/wheels.urdf.xacro" />
@@ -61,5 +62,5 @@
     <origin xyz="${front_wheel_L} 0 0" rpy="0 0 0" />
   </xacro:front_wheel>
-  <!-- Sensors -->
+  <!-- IMU -->
   <link name="imu_link">
     <visual><geometry><sphere radius="0.0025"/></geometry></visual>
@@ -70,3 +71,16 @@
     <child link="imu_link" />
   </joint>
+  <!-- Infrared Marker -->
+  <xacro:if value="${use_smocap_ir_marker}">
+    <xacro:cs_smocap_ir_marker>
+      <origin xyz="0 0 0.06" rpy="0 0 0" />
+    </xacro:cs_smocap_ir_marker>
+  </xacro:if>
+  <!-- Camera -->
+  <xacro:if value="${use_eachine_camera}">
+    <xacro:property name="cam_look_down_deg" value="25." />
+    <xacro:cs_camera_eachine>
+      <origin xyz="0.09 0 0.04" rpy="0 ${cam_look_down_deg/180*pi}} 0" />
+    </xacro:cs_camera_eachine>
+  </xacro:if>
 </robot>

File: oscar/oscar_description/urdf/oscar_v0.urdf.xacro (robot description, xacro)
@@ -1,5 +1,8 @@
 <?xml version="1.0"?>
 <robot name="oscar" xmlns:xacro="http://www.ros.org/wiki/xacro">
+  <xacro:property name="use_eachine_camera" value="False" />
+  <xacro:property name="use_smocap_ir_marker" value="True" />
   <xacro:property name="high_definition_wheel_visual" value="True" />
+  <xacro:property name="high_definition_camera_visual" value="True" />
   <xacro:include filename="$(find oscar_description)/urdf/oscar.urdf.xacro" />
 </robot>

File: oscar_simulator/oscar_gazebo/urdf/oscar.gazebo.urdf.xacro (robot description, xacro)
@@ -3,4 +3,5 @@
   <xacro:property name="robot_name" default="oscar_v0" />
   <xacro:include filename="$(find oscar_description)/urdf/${robot_name}.urdf.xacro" />
+  <xacro:include filename="$(find common_simulations)/urdf/sensors_gazebo.urdf.xacro" />
   <xacro:property name="wheel_mu1" default="10000" />
   <xacro:property name="wheel_mu2" default="10000" />
@@ -10,4 +11,5 @@
   <gazebo reference="front_axle_carrier_link"><material>Gazebo/Blue</material></gazebo>
   <gazebo reference="imu_link"><material>Gazebo/Red</material></gazebo>
+  <gazebo reference="camera_link"><material>Gazebo/Red</material></gazebo>
   <gazebo reference="left_wheel_link">
     <mu1>${wheel_mu1}</mu1>
@@ -79,4 +81,8 @@
   </gazebo>
   -->
+ <!-- Camera -->
+ <xacro:if value="${use_eachine_camera}">
+   <xacro:gazebo_eachine_camera cam_name="camera1"/>
+ </xacro:if>
   <!-- Ground Truth  -->
   <gazebo>

Commit message: a

File: oscar/oscar_description/urdf/oscar.urdf.xacro (robot description, xacro)
@@ -14,5 +14,5 @@
   <xacro:property name="rear_wheel_axle_joint_eff_limit" value="10.0" />
   <xacro:property name="rear_wheel_axle_joint_vel_limit" value="20.0" />
-  <xacro:property name="rear_wheel_joint_damping"  value="0.01" />
+  <xacro:property name="rear_wheel_joint_damping"  value="0.05" />
   <xacro:property name="rear_wheel_joint_friction" value="0.01" />
   <xacro:property name="front_wheel_radius"  value="0.03" />
@@ -73,5 +73,5 @@
   <!-- Infrared Marker -->
   <xacro:if value="${use_smocap_ir_marker}">
-    <xacro:cs_smocap_ir_marker>
+    <xacro:cs_smocap_ir_marker mesh="${smocap_ir_marker_mesh}">
       <origin xyz="0 0 0.06" rpy="0 0 0" />
     </xacro:cs_smocap_ir_marker>
