Commit message: bbb/jetson coms

File: oscar/oscar_description/urdf/christine_v0.urdf.xacro (robot description, xacro)
@@ -2,5 +2,9 @@
 <robot name="oscar" xmlns:xacro="http://www.ros.org/wiki/xacro">
   <!--<xacro:include filename="$(find oscar_description)/urdf/oscar_defaults.urdf.xacro" /> -->
-  <xacro:property name="use_eachine_camera" value="False" />
+  <xacro:property name="use_camera" value="true" />
+  <xacro:property name="cam_name" value="camera_road_front" />
+  <xacro:property name="cam_hd_visual" value="true" />
+  <xacro:property name="cam_cl_to_ref_xyz" value="0.19881951 -0.00770707  0.13167937" />
+  <xacro:property name="cam_cl_to_ref_rpy" value="0.02039069  0.35225342  0.06052593" />
   <xacro:property name="use_smocap_ir_marker" value="False" />
   <xacro:property name="high_definition_wheel_visual" value="True" />

File: oscar/oscar_description/urdf/oscar.urdf.xacro (robot description, xacro)
@@ -33,4 +33,10 @@
   <!-- Body -->
   <link name="base_link"></link>
+  <link name="base_link_footprint"></link>
+  <joint name="base_link_footprint_joint" type="fixed">
+    <origin xyz="0 0 ${-left_wheel_radius}" rpy="0 0 0" />
+    <parent link="base_link"/>
+    <child link="base_link_footprint" />
+  </joint>
   <link name="chassis_link">
     <visual>
@@ -78,8 +84,15 @@
   </xacro:if>
   <!-- Camera -->
-  <xacro:if value="${use_eachine_camera}">
-    <xacro:property name="cam_look_down_deg" value="25." />
-    <xacro:cs_camera_eachine>
-      <origin xyz="0.09 0 0.04" rpy="0 ${cam_look_down_deg/180*pi}} 0" />
+  <!-- <xacro:if value="${use_eachine_camera}"> -->
+  <!--   <xacro:property name="cam_look_down_deg" value="25." /> -->
+  <!--   <xacro:cs_camera_eachine> -->
+  <!--     <origin xyz="0.09 0 0.04" rpy="0 ${cam_look_down_deg/180*pi}} 0" /> -->
+  <!--   </xacro:cs_camera_eachine> -->
+  <!-- </xacro:if> -->
+  <!-- Camera -->
+  <xacro:include filename="$(find common_robots)/urdf/sensors.urdf.xacro" />
+  <xacro:if value="${use_camera}">
+    <xacro:cs_camera_eachine cam_name="${cam_name}" origin_ref_frame="base_link_footprint">
+      <origin xyz="${cam_cl_to_ref_xyz}" rpy="${cam_cl_to_ref_rpy}" />
     </xacro:cs_camera_eachine>
   </xacro:if>

Commit message: improving christine model; working toward simulation

File: oscar/oscar_description/urdf/christine_v0.urdf.xacro (robot description, xacro)
@@ -1,12 +1,29 @@
 <?xml version="1.0"?>
 <robot name="oscar" xmlns:xacro="http://www.ros.org/wiki/xacro">
-  <!--<xacro:include filename="$(find oscar_description)/urdf/oscar_defaults.urdf.xacro" /> -->
+  <xacro:include filename="$(find oscar_description)/urdf/oscar_defaults.urdf.xacro" />
+  <xacro:property name="chassis_length" value="0.08" />
+  <xacro:property name="chassis_width"  value="0.065" />
+  <xacro:property name="chassis_height" value="0.01" />
+  <xacro:property name="chassis_mass"   value="0.20" />
+  <xacro:property name="chassis_dx"     value="0.04" />
+  <xacro:property name="left_wheel_radius"  value="0.04" />
+  <xacro:property name="right_wheel_radius" value="0.04" />
+  <xacro:property name="wheel_track"   value="0.205" />
+  <xacro:property name="wheel_width"  value="0.04" />
+  <xacro:property name="front_wheel_radius"  value="0.04" />
+  <xacro:property name="front_wheel_L" value="0.27" />
+  <xacro:property name="front_wheel_width"   value="0.03" />
   <xacro:property name="use_camera" value="true" />
   <xacro:property name="cam_name" value="camera_road_front" />
   <xacro:property name="cam_hd_visual" value="true" />
-  <xacro:property name="cam_cl_to_ref_xyz" value="0.19881951 -0.00770707  0.13167937" />
-  <xacro:property name="cam_cl_to_ref_rpy" value="0.02039069  0.35225342  0.06052593" />
+  <!-- initial wood mount -->
+  <!-- <xacro:property name="cam_cl_to_ref_xyz" value="0.19881951 -0.00770707  0.13167937" /> -->
+  <!-- <xacro:property name="cam_cl_to_ref_rpy" value="0.02039069  0.35225342  0.06052593" /> -->
+  <!-- new printed mount -->
+  <xacro:property name="cam_cl_to_ref_xyz" value="0.24041413  0.00764807  0.17355088" />
+  <xacro:property name="cam_cl_to_ref_rpy" value="-4.83558341e-04   5.51295376e-01   4.91191358e-02" />
+  <xacro:property name="use_eachine_camera" value="false"/>
   <xacro:property name="use_smocap_ir_marker" value="False" />
-  <xacro:property name="high_definition_wheel_visual" value="True" />
+  <xacro:property name="high_definition_wheel_visual"  value="True" />
   <xacro:property name="high_definition_camera_visual" value="True" />
   <xacro:include filename="$(find oscar_description)/urdf/oscar.urdf.xacro" />

File: oscar/oscar_description/urdf/oscar.urdf.xacro (robot description, xacro)
@@ -1,28 +1,5 @@
 <?xml version="1.0"?>
 <robot name="oscar" xmlns:xacro="http://www.ros.org/wiki/xacro">
-  <xacro:property name="chassis_length" value="0.08" />
-  <xacro:property name="chassis_width"  value="0.065" />
-  <xacro:property name="chassis_height" value="0.01" />
-  <xacro:property name="chassis_mass"   value="0.20" />
-  <xacro:property name="chassis_dx"     value="0.04" />
-  <xacro:property name="left_wheel_radius"  value="0.03" />
-  <xacro:property name="right_wheel_radius" value="0.03" />
-  <xacro:property name="wheel_width"  value="0.02" />
-  <xacro:property name="wheel_track"  value="0.09" />
-  <xacro:property name="wheel_mass"   value="0.02" />
-  <xacro:property name="steering_servo_no_load_speed" value="2.5" />
-  <xacro:property name="rear_wheel_axle_joint_eff_limit" value="10.0" />
-  <xacro:property name="rear_wheel_axle_joint_vel_limit" value="20.0" />
-  <xacro:property name="rear_wheel_joint_damping"  value="0.05" />
-  <xacro:property name="rear_wheel_joint_friction" value="0.01" />
-  <xacro:property name="front_wheel_radius"  value="0.03" />
-  <xacro:property name="front_wheel_L"       value="0.08" />
-  <xacro:property name="front_wheel_width"   value="0.02" />
-  <xacro:property name="steering_servo_stall_torque" value="10.0" />
-  <xacro:property name="steering_servo_no_load_speed" value="2.5" />
-  <xacro:property name="front_wheel_axle_joint_eff_limit" value="10.0" />
-  <xacro:property name="front_wheel_axle_joint_vel_limit" value="20.0" />
-  <xacro:property name="front_wheel_axle_joint_damping"  value="0.00001" />
-  <xacro:property name="front_wheel_axle_joint_friction" value="0.00001" />
+  <!-- see oscar_defaults.urdf.xacro for parameters expected by this model -->
   <!-- Common macros -->
   <xacro:include filename="$(find common_robots)/urdf/inertias.urdf.xacro" />

File: oscar/oscar_description/urdf/oscar_v0.urdf.xacro (robot description, xacro)
@@ -1,6 +1,9 @@
 <?xml version="1.0"?>
 <robot name="oscar" xmlns:xacro="http://www.ros.org/wiki/xacro">
+  <xacro:include filename="$(find oscar_description)/urdf/oscar_defaults.urdf.xacro" />
+  <xacro:property name="use_camera" value="False" />
   <xacro:property name="use_eachine_camera" value="False" />
   <xacro:property name="use_smocap_ir_marker" value="True" />
+  <xacro:property name="smocap_ir_marker_mesh" value="ir_marker_0.dae" />
   <xacro:property name="high_definition_wheel_visual" value="True" />
   <xacro:property name="high_definition_camera_visual" value="True" />

Commit message: updated christine extrinsic calibration

File: oscar/oscar_description/urdf/christine_v0.urdf.xacro (robot description, xacro)
@@ -21,6 +21,9 @@
   <!-- <xacro:property name="cam_cl_to_ref_rpy" value="0.02039069  0.35225342  0.06052593" /> -->
   <!-- new printed mount -->
-  <xacro:property name="cam_cl_to_ref_xyz" value="0.24041413  0.00764807  0.17355088" />
-  <xacro:property name="cam_cl_to_ref_rpy" value="-4.83558341e-04   5.51295376e-01   4.91191358e-02" />
+  <!-- before sept 30 2019 -->
+  <!-- <xacro:property name="cam_cl_to_ref_xyz" value="0.24041413  0.00764807  0.17355088" /> -->
+  <!-- <xacro:property name="cam_cl_to_ref_rpy" value="-4.83558341e-04   5.51295376e-01   4.91191358e-02" /> -->
+  <xacro:property name="cam_cl_to_ref_xyz" value=" 0.21862012 -0.00555091  0.16551083" />
+  <xacro:property name="cam_cl_to_ref_rpy" value="-0.0208105   0.51668558  0.03265788" />
   <xacro:property name="use_eachine_camera" value="false"/>
   <xacro:property name="use_smocap_ir_marker" value="False" />

Commit message: added horizon camera

File: oscar/oscar_description/urdf/christine_v0.urdf.xacro (robot description, xacro)
@@ -26,4 +26,9 @@
   <xacro:property name="cam_cl_to_ref_xyz" value=" 0.21862012 -0.00555091  0.16551083" />
   <xacro:property name="cam_cl_to_ref_rpy" value="-0.0208105   0.51668558  0.03265788" />
+  <!-- Camera horizon -->
+  <xacro:property name="use_camera2" value="true" />
+  <xacro:property name="cam2_name" value="camera_horiz_front" />
+  <xacro:property name="cam2_cl_to_ref_xyz" value="0.06483087  0.00032532  0.22" />
+  <xacro:property name="cam2_cl_to_ref_rpy" value="0.0077082   -0.1  0.02633946" />
   <xacro:property name="use_eachine_camera" value="false"/>
   <xacro:property name="use_smocap_ir_marker" value="False" />

File: oscar/oscar_description/urdf/oscar.urdf.xacro (robot description, xacro)
@@ -74,3 +74,8 @@
     </xacro:cs_camera_eachine>
   </xacro:if>
+  <xacro:if value="${use_camera2}">
+    <xacro:cs_camera_eachine cam_name="${cam2_name}" origin_ref_frame="base_link_footprint">
+      <origin xyz="${cam2_cl_to_ref_xyz}" rpy="${cam2_cl_to_ref_rpy}" />
+    </xacro:cs_camera_eachine>
+  </xacro:if>
 </robot>

Commit message: calibrated christine camera

File: oscar/oscar_description/urdf/christine_v0.urdf.xacro (robot description, xacro)
@@ -24,6 +24,10 @@
   <!-- <xacro:property name="cam_cl_to_ref_xyz" value="0.24041413  0.00764807  0.17355088" /> -->
   <!-- <xacro:property name="cam_cl_to_ref_rpy" value="-4.83558341e-04   5.51295376e-01   4.91191358e-02" /> -->
-  <xacro:property name="cam_cl_to_ref_xyz" value=" 0.21862012 -0.00555091  0.16551083" />
-  <xacro:property name="cam_cl_to_ref_rpy" value="-0.0208105   0.51668558  0.03265788" />
+  <!-- calib enac z -->
+  <!-- <xacro:property name="cam_cl_to_ref_xyz" value=" 0.21862012 -0.00555091  0.16551083" /> -->
+  <!-- <xacro:property name="cam_cl_to_ref_rpy" value="-0.0208105   0.51668558  0.03265788" /> -->
+  <!-- guesdes -->
+  <xacro:property name="cam_cl_to_ref_xyz" value=" 2.29319801e-01,   2.27515078e-04,   1.62087062e-01" />
+  <xacro:property name="cam_cl_to_ref_rpy" value="-0.01986798,  0.52218905,  0.05208673" />
   <!-- Camera horizon -->
   <xacro:property name="use_camera2" value="true" />

Commit message: swapped camera after crash

File: oscar/oscar_description/urdf/christine_v0.urdf.xacro (robot description, xacro)
@@ -28,6 +28,9 @@
   <!-- <xacro:property name="cam_cl_to_ref_rpy" value="-0.0208105   0.51668558  0.03265788" /> -->
   <!-- guesdes -->
-  <xacro:property name="cam_cl_to_ref_xyz" value=" 2.29319801e-01,   2.27515078e-04,   1.62087062e-01" />
-  <xacro:property name="cam_cl_to_ref_rpy" value="-0.01986798,  0.52218905,  0.05208673" />
+  <!-- <xacro:property name="cam_cl_to_ref_xyz" value=" 2.29319801e-01,   2.27515078e-04,   1.62087062e-01" /> -->
+  <!-- <xacro:property name="cam_cl_to_ref_rpy" value="-0.01986798,  0.52218905,  0.05208673" /> -->
+  <!-- enac z 4 -->
+  <xacro:property name="cam_cl_to_ref_xyz" value=" 0.21262579,  0.00281551,  0.15738715" />
+  <xacro:property name="cam_cl_to_ref_rpy" value="-0.03868774,  0.56221351, -0.04609374" />
   <!-- Camera horizon -->
   <xacro:property name="use_camera2" value="true" />
